File: IMU 9DoF AHRS.brd (EAGLE design)
At the start: 46.5 x 26.7 mm, 49 parts, among them IC1 ATMEGA328P, J2 AVR_SPI_PRG_6PTH, U1 ADP122AUJZ-3.3-R7, U3 MPL3115A2LGA8, U4 HTU21DSMD, U5 EM406, Y1 8MHZ

Commit message: updated EAGLE files to latest revision
updated EAGLE files to latest revision
added Schematic in PDF format
updated Gerber Data
Parts:
- C10: device SparkFun-Capacitors:1206 -> SparkFun-Capacitors:0805
- R3, R4: value 4.7K -> 2.2K
- moved R3 3.05 mm to (24.6, 13.5)
- moved R4 3.05 mm to (21.6, 13.5)
Connections:
- removed net A6: IC1.19
- removed net A7: IC1.22
- removed net XBEE-RTS: U$1.16
- net SCL: now also U3.8; no longer U3.7
- net SDA: now also U3.7; no longer U3.8
- net VCC: no longer U5.2
- net VIN: now also U5.2
Routing:
- net VIN: track 46.7 -> 98.6 mm, vias 0 -> 2
- net XBEE-RTS: track 3.48 -> 0.00 mm, vias 1 -> 0
- net SCL: track 36.4 -> 33.6 mm
- net VCC: track 47.4 -> 44.6 mm, vias 14 -> 13
- net RESET: track 66.0 -> 63.3 mm
- net SDA: track 36.2 -> 38.2 mm
- net GND: vias 15 -> 16
Other:
- board text added: "2.2K"
- board text added: "XBee"
- board text removed: "4.7K"
